File: schematics/picotouch.brd (EAGLE design)
At the start: 250 x 34 mm, 47 parts, among them U1 RASPBERRY_PICOSMD-TH

Commit message: submitted to pcbway
Parts:
- added U$1: (no value), todstuff:PICOTOUCH_TOPSILK
- moved R18 18.1 mm to (166.7, 7.00)
- moved R20 18.1 mm to (166.7, 25.0)
- moved TP18 18.0 mm to (174.5, 7.00)
- moved TP20 18.0 mm to (174.5, 25.0)
- moved R21 18.0 mm to (193.7, 7.00)
- moved TP23 18.0 mm to (185.5, 25.0)
- moved R23 18.0 mm to (193.2, 25.0)
- moved TP21 18.0 mm to (185.5, 7.00)
- moved R19 1.50 mm to (166.7, 16.0)
- moved TP19 0.73 mm to (174.5, 16.0)
- moved TP22 0.50 mm to (185.5, 16.0)
Routing:
- net GP0: track 0.00 -> 264.9 mm, vias 0 -> 1
- net GP1: track 0.00 -> 241.5 mm, vias 0 -> 1
- net GP2: track 0.00 -> 237.9 mm, vias 0 -> 1
- net GP4: track 0.00 -> 237.5 mm
- net GP3: track 0.00 -> 217.6 mm, vias 0 -> 1
- net GP5: track 0.00 -> 197.6 mm, vias 0 -> 1
- net GP7: track 0.00 -> 174.8 mm, vias 0 -> 1
- net GP6: track 0.00 -> 171.9 mm, vias 0 -> 1
- net GP11: track 0.00 -> 156.3 mm
- net GP9: track 0.00 -> 153.3 mm, vias 0 -> 1
- net GP8: track 0.00 -> 151.2 mm, vias 0 -> 1
- net GP12: track 0.00 -> 137.1 mm
- net GND: track 0.00 -> 136.9 mm
- net GP10: track 0.00 -> 127.3 mm, vias 0 -> 1
- net GP14: track 0.00 -> 101.3 mm, vias 0 -> 1
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Other:
- outline, holes or cut-outs redrawn
- board text added: "20210413 - @todbot"
- board text added: "all resistors are 1M"
- board text added: "github.com/todbot/picotouch"
- board text added: "works with CircuitPython!"
