File: schematics/picotouchsynth.brd (EAGLE design)
At the start: 207 x 49.5 mm, 74 parts, among them IC1 H11L1MS, J1 SJ-3523-SMT, J2 SJ-3523-SMT, U1 RASPBERRY_PICOSMD-TH

Commit message: more picotouchsynth
Parts:
- moved C1 132.1 mm to (138.4, 30.5), turned to 90 degrees
- moved LED1 124.5 mm to (134.6, 30.5), turned to 270 degrees
- moved LED13 124.5 mm to (10.2, 30.5), turned to 270 degrees
- moved R1 124.5 mm to (134.6, 17.8)
- moved R13 124.5 mm to (10.2, 17.8)
- moved TP1 124.5 mm to (134.6, 7.62)
- moved TP13 124.5 mm to (10.2, 7.62)
- moved C13 116.8 mm to (14.0, 30.5), turned to 90 degrees
- moved C2 105.4 mm to (120.7, 30.5), turned to 90 degrees
- moved TP12 98.6 mm to (19.1, 20.3)
- moved TP2 98.6 mm to (116.8, 7.62)
- moved R12 98.1 mm to (19.1, 10.2), turned to 270 degrees
- moved R2 98.1 mm to (116.8, 17.8), turned to 90 degrees
- moved LED12 97.8 mm to (19.1, 30.5), turned to 270 degrees
- moved LED2 97.8 mm to (116.8, 30.5), turned to 270 degrees
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- renumbered R20 to R444, R21 to R555, R22 to R333, R23 to R222, R24 to R111, R25 to R666, R26 to R777
Connections:
- removed net T0: R1.1, TP1.TP, U1.20, U1.P$20
- new net LED_DATA: LED1.4-DIN, U1.21, U1.P$21
- new net T16: R16.1, TP16.TP, U1.20, U1.P$20
- net T1: now also R1.1, TP1.TP, U1.1, U1.P$1; no longer R2.1, TP2.TP, U1.19, U1.P$19
- net T10: now also R10.1, TP10.TP, U1.12, U1.P$12; no longer R11.1, TP11.TP, U1.7, U1.P$7
- net T11: now also R11.1, TP11.TP, U1.14, U1.P$14; no longer R12.1, TP12.TP, U1.6, U1.P$6
- net T12: now also R12.1, TP12.TP, U1.15, U1.P$15; no longer R13.1, TP13.TP, U1.5, U1.P$5
- net T13: now also R13.1, TP13.TP, U1.16, U1.P$16; no longer R14.1, TP14.TP, U1.4, U1.P$4
- net T14: now also R14.1, TP14.TP, U1.17, U1.P$17; no longer R15.1, TP15.TP, U1.2, U1.P$2
- net T15: now also R15.1, TP15.TP, U1.19, U1.P$19; no longer R16.1, TP16.TP, U1.1, U1.P$1
- net T2: now also R2.1, TP2.TP, U1.2, U1.P$2; no longer R3.1, TP3.TP, U1.17, U1.P$17
- net T3: now also R3.1, TP3.TP, U1.4, U1.P$4; no longer R4.1, TP4.TP, U1.16, U1.P$16
- net T4: now also R4.1, TP4.TP, U1.5, U1.P$5; no longer R5.1, TP5.TP, U1.15, U1.P$15
- net T5: now also R5.1, TP5.TP, U1.6, U1.P$6; no longer R6.1, TP6.TP, U1.14, U1.P$14
- net T6: now also R6.1, TP6.TP, U1.7, U1.P$7; no longer R7.1, TP7.TP, U1.12, U1.P$12
- net T7: now also R7.1, TP7.TP, U1.9, U1.P$9; no longer R8.1, TP8.TP, U1.11, U1.P$11
- net T8: now also R8.1, TP8.TP; no longer R9.1, TP9.TP
- net T9: now also R9.1, TP9.TP, U1.11, U1.P$11; no longer R10.1, TP10.TP, U1.9, U1.P$9
Routing:
- net T0: track 161.6 -> 0.00 mm, vias 1 -> 0
- net T12: track 84.2 -> 172.9 mm
- net T16: track 0.00 -> 82.0 mm, vias 0 -> 2
- net +3V3: track 188.0 -> 120.4 mm
- net T1: track 161.7 -> 98.6 mm, vias 1 -> 2
- net T15: track 165.8 -> 104.2 mm
- net T11: track 100.5 -> 161.3 mm
- net T13: track 118.1 -> 174.3 mm, vias 2 -> 1
- net T10: track 110.0 -> 163.4 mm
- net LED_DATA: track 0.00 -> 43.3 mm, vias 0 -> 1
- net T2: track 152.7 -> 109.7 mm
- net T9: track 110.9 -> 151.8 mm
- net T3: track 152.0 -> 116.5 mm
- net T8: track 120.9 -> 150.4 mm
- net T7: track 123.1 -> 146.2 mm
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