File: schematics/picotouchsynth.sch (EAGLE design)
At the start: 74 parts, among them IC1 H11L1MS, J1 SJ-3523-SMT, J2 SJ-3523-SMT, U1 RASPBERRY_PICOSMD-TH

Commit message: more picotouchsynth
Parts:
- renumbered R20 to R444, R21 to R555, R22 to R333, R23 to R222, R24 to R111, R25 to R666, R26 to R777
Connections:
- removed net T0: R1.1, TP1.TOUCH, U1.GP15
- new net LED_DATA: LED1.DI, U1.GP16
- new net T16: R16.1, TP16.TOUCH, U1.GP15
- net T1: now also R1.1, TP1.TOUCH, U1.GP0; no longer R2.1, TP2.TOUCH, U1.GP14
- net T10: now also R10.1, TP10.TOUCH, U1.GP9; no longer R11.1, TP11.TOUCH, U1.GP5
- net T11: now also R11.1, TP11.TOUCH, U1.GP10; no longer R12.1, TP12.TOUCH, U1.GP4
- net T12: now also R12.1, TP12.TOUCH, U1.GP11; no longer R13.1, TP13.TOUCH, U1.GP3
- net T13: now also R13.1, TP13.TOUCH, U1.GP12; no longer R14.1, TP14.TOUCH, U1.GP2
- net T14: now also R14.1, TP14.TOUCH, U1.GP13; no longer R15.1, TP15.TOUCH, U1.GP1
- net T15: now also R15.1, TP15.TOUCH, U1.GP14; no longer R16.1, TP16.TOUCH, U1.GP0
- net T2: now also R2.1, TP2.TOUCH, U1.GP1; no longer R3.1, TP3.TOUCH, U1.GP13
- net T3: now also R3.1, TP3.TOUCH, U1.GP2; no longer R4.1, TP4.TOUCH, U1.GP12
- net T4: now also R4.1, TP4.TOUCH, U1.GP3; no longer R5.1, TP5.TOUCH, U1.GP11
- net T5: now also R5.1, TP5.TOUCH, U1.GP4; no longer R6.1, TP6.TOUCH, U1.GP10
- net T6: now also R6.1, TP6.TOUCH, U1.GP5; no longer R7.1, TP7.TOUCH, U1.GP9
- net T7: now also R7.1, TP7.TOUCH, U1.GP6; no longer R8.1, TP8.TOUCH, U1.GP8
- net T8: now also R8.1, TP8.TOUCH; no longer R9.1, TP9.TOUCH
- net T9: now also R9.1, TP9.TOUCH, U1.GP8; no longer R10.1, TP10.TOUCH, U1.GP6
Other:
- moved on the sheet: R1, R10, R11, R12, R13, R14, R15, R16, R2, R3, R4, R5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

Commit message: picotouchsynth version sent to fab
Parts:
- removed C22: 100n, rcl:C-EUC0805
- added C16: 100n, rcl:C-EUC0805
- C14: value (none) -> 100n
- renumbered C21 to C15, R111 to R17, R222 to R18, R333 to R19, R444 to R20, R555 to R21, R666 to R22, R777 to R23
Connections:
- net +3V3: now also C16.1; no longer C14.1
- net GND: now also C16.2; no longer C22.2
- net N$48: now also C14.1; no longer C22.1
Other:
- note added: "OLED is mounted on bottom of PCB"
- moved on the sheet: C14
