File: schematics/picotouch_synth.sch (EAGLE design)
At the start: 100 parts, among them IC2 H11L1MS, J1 AUDIO-JACK-TRRS, J3 AUDIO-JACK-TRRS, J4 AUDIO-JACK-TRRS, U1 RASPBERRY_PICOSMD

Commit message: first cut at picotouch_synth pcb art
Parts:
- R1, R11, R12, R13, R14, R15, R16, R17, R18, R19, R2, R20, R21, R22, R3, R4, R5, R6, R7, R8, R9: value (none) -> 1M
