File: schematics/picotouch_grid/picotouch_grid.sch (EAGLE design)
At the start: 140 parts, among them J3 AUDIO-JACK-TRRS, K1 TOUCHKEYH, K10 TOUCHKEYH, K11 TOUCHKEYH, K12 TOUCHKEYH, K13 TOUCHKEYH, K14 TOUCHKEYH, K15 TOUCHKEYH, K16 TOUCHKEYH, K17 TOUCHKEYH, K18 TOUCHKEYH, K19 TOUCHKEYH, K2 TOUCHKEYH, K20 TOUCHKEYH, K21 TOUCHKEYH, K22 TOUCHKEYH, K23 TOUCHKEYH, K24 TOUCHKEYH, K25 TOUCHKEYH, K26 TOUCHKEYH, K27 TOUCHKEYH, K28 TOUCHKEYH, K29 TOUCHKEYH, K3 TOUCHKEYH, K30 TOUCHKEYH, K31 TOUCHKEYH, K32 TOUCHKEYH, K33 TOUCHKEYH, K34 TOUCHKEYH, K35 TOUCHKEYH, K36 TOUCHKEYH, K37 TOUCHKEYH, K38 TOUCHKEYH, K39 TOUCHKEYH, K4 TOUCHKEYH, K40 TOUCHKEYH, K5 TOUCHKEYH, K6 TOUCHKEYH, K7 TOUCHKEYH, K8 TOUCHKEYH, K9 TOUCHKEYH, U1 RASPBERRY_PICOSMD

Commit message: reorg grid idea
Parts:
- removed J3: AUDIO-JACK-TRRS, audio_jacks_todbot:AUDIO-JACK-TRRS
- added DISP1: (no value), SparkFun-Connectors:CONN_04
- J1: value (none) -> AUDIO-JACK-TRRS; device SparkFun-Connectors:CONN_04 -> audio_jacks_todbot:AUDIO-JACK-TRRS; LCSC (none) -> C431535
- LED1: LCSC (none) -> C5149201
- renumbered CONN1 to J2
Connections:
- net +3V3: now also DISP1.2; no longer J1.2
- net GND: now also DISP1.1, J1.EARTH; no longer J1.1, J3.EARTH
- net N$38: now also J1.RING1; no longer J3.RING1
- net N$8: now also J1.TIP; no longer J3.TIP
- net SCL: now also DISP1.3; no longer J1.3
- net SDA: now also DISP1.4; no longer J1.4
Other:
- note added: "7 Feb 2023 - @todbot / Tod Kurt"

Commit message: added gpio pins 16,17,18,19 as smd touchpads for hacking
Parts:
- added 16, 17, 18, 19: TPTP15R, testpad:TPTP15R
Connections:
- new net N$39: 16.TP, U1.GP16
- new net N$40: 17.TP, U1.GP17
- new net N$41: 18.TP, U1.GP18
- new net N$42: 19.TP, U1.GP19

Commit message: added test points
Parts:
- added 3V3, 3VM, GND, M, NEOPIXEL: TPTP15R, testpad:TPTP15R
Connections:
- net +3V3: now also 3V3.TP
- net GND: now also GND.TP
- net N$38: now also 3VM.TP
- net N$8: now also M.TP
- net NEOPIXEL: now also NEOPIXEL.TP
Changed lines of the file:
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@@
 <part name="18" library="testpad" library_urn="urn:adsk.eagle:library:385" deviceset="TP" device="TP15R" package3d_urn="urn:adsk.eagle:package:27968/1" value="TPTP15R"/>
 <part name="19" library="testpad" library_urn="urn:adsk.eagle:library:385" deviceset="TP" device="TP15R" package3d_urn="urn:adsk.eagle:package:27968/1" value="TPTP15R"/>
+<part name="3V3" library="testpad" library_urn="urn:adsk.eagle:library:385" deviceset="TP" device="TP15R" package3d_urn="urn:adsk.eagle:package:27968/1" value="TPTP15R"/>
+<part name="+3V86" library="supply1" library_urn="urn:adsk.eagle:library:371" deviceset="+3V3" device=""/>
+<part name="GND" library="testpad" library_urn="urn:adsk.eagle:library:385" deviceset="TP" device="TP15R" package3d_urn="urn:adsk.eagle:package:27968/1" value="TPTP15R"/>
+<part name="GND2" library="supply1" library_urn="urn:adsk.eagle:library:371" deviceset="GND" device=""/>
+<part name="NEOPIXEL" library="testpad" library_urn="urn:adsk.eagle:library:385" deviceset="TP" device="TP15R" package3d_urn="urn:adsk.eagle:package:27968/1" value="TPTP15R"/>
+<part name="3VM" library="testpad" library_urn="urn:adsk.eagle:library:385" deviceset="TP" device="TP15R" package3d_urn="urn:adsk.eagle:package:27968/1" value="TPTP15R"/>
+<part name="M" library="testpad" library_urn="urn:adsk.eagle:library:385" deviceset="TP" device="TP15R" package3d_urn="urn:adsk.eagle:package:27968/1" value="TPTP15R"/>
 </parts>
 <sheets>
@@
 <attribute name="TP_SIGNAL_NAME" x="156.21" y="186.69" size="1.778" layer="97" rot="R270"/>
 </instance>
+<instance part="3V3" gate="G$1" x="45.72" y="231.14" smashed="yes" rot="R90">
+<attribute name="NAME" x="44.45" y="232.41" size="1.778" layer="95" rot="R180"/>
+<attribute name="TP_SIGNAL_NAME" x="46.99" y="232.41" size="1.778" layer="97" rot="R90"/>
+</instance>
+<instance part="+3V86" gate="G$1" x="50.8" y="231.14" smashed="yes" rot="R270">
+<attribute name="VALUE" x="57.658" y="232.156" size="1.778" layer="96" rot="R180"/>
+</instance>
+<instance part="GND" gate="G$1" x="45.72" y="220.98" smashed="yes" rot="R90">
+<attribute name="NAME" x="44.45" y="219.71" size="1.778" layer="95" rot="R90"/>
+<attribute name="TP_SIGNAL_NAME" x="46.99" y="222.25" size="1.778" layer="97" rot="R90"/>
+</instance>
+<instance part="GND2" gate="1" x="50.8" y="220.98" smashed="yes" rot="R90">
+<attribute name="VALUE" x="53.34" y="218.44" size="1.778" layer="96" rot="R90"/>
+</instance>
+<instance part="NEOPIXEL" gate="G$1" x="45.72" y="226.06" smashed="yes" rot="R90">
+<attribute name="NAME" x="44.45" y="227.33" size="1.778" layer="95" rot="R180"/>
+<attribute name="TP_SIGNAL_NAME" x="46.99" y="227.33" size="1.778" layer="97" rot="R90"/>
+</instance>
+<instance part="3VM" gate="G$1" x="53.34" y="127" smashed="yes" rot="R180">
+<attribute name="NAME" x="52.07" y="125.73" size="1.778" layer="95" rot="R270"/>
+<attribute name="TP_SIGNAL_NAME" x="52.07" y="128.27" size="1.778" layer="97" rot="R180"/>
+</instance>
+<instance part="M" gate="G$1" x="53.34" y="154.94" smashed="yes">
+<attribute name="NAME" x="54.61" y="156.21" size="1.778" layer="95" rot="R90"/>
+<attribute name="TP_SIGNAL_NAME" x="54.61" y="153.67" size="1.778" layer="97"/>
+</instance>
 </instances>
 <busses>
@@
 <junction x="60.96" y="208.28"/>
 </segment>
+<segment>
+<pinref part="GND" gate="G$1" pin="TP"/>
+<pinref part="GND2" gate="1" pin="GND"/>
+</segment>
 </net>
 <net name="+3V3" class="0">
@@
 <pinref part="J2" gate="G$1" pin="V+"/>
 <wire x1="58.42" y1="205.74" x2="48.26" y2="205.74" width="0.1524" layer="91"/>
+</segment>
+<segment>
+<pinref part="3V3" gate="G$1" pin="TP"/>
+<pinref part="+3V86" gate="G$1" pin="+3V3"/>
 </segment>
 </net>
@@
 <segment>
 <pinref part="U1" gate="U$1" pin="GP28"/>
-<wire x1="147.32" y1="210.82" x2="160.02" y2="210.82" width="0.1524" layer="91"/>
+<wire x1="147.32" y1="210.82" x2="162.56" y2="210.82" width="0.1524" layer="91"/>
 <label x="152.4" y="210.82" size="1.778" layer="95"/>
+</segment>
+<segment>
+<pinref part="NEOPIXEL" gate="G$1" pin="TP"/>
+<wire x1="48.26" y1="226.06" x2="55.88" y2="226.06" width="0.1524" layer="91"/>
+<label x="55.88" y="226.06" size="1.778" layer="95"/>
 </segment>
 </net>
@@
 <segment>
 <pinref part="J1" gate="G$1" pin="TIP"/>
-<wire x1="66.04" y1="144.78" x2="50.8" y2="144.78" width="0.1524" layer="91"/>
+<wire x1="66.04" y1="144.78" x2="53.34" y2="144.78" width="0.1524" layer="91"/>
 <pinref part="R16" gate="G$1" pin="1"/>
+<pinref part="M" gate="G$1" pin="TP"/>
+<wire x1="53.34" y1="144.78" x2="50.8" y2="144.78" width="0.1524" layer="91"/>
+<wire x1="53.34" y1="152.4" x2="53.34" y2="144.78" width="0.1524" layer="91"/>
+<junction x="53.34" y="144.78"/>
 </segment>
 </net>
@@
 <pinref part="R15" gate="G$1" pin="1"/>
 <wire x1="55.88" y1="139.7" x2="55.88" y2="137.16" width="0.1524" layer="91"/>
-<wire x1="55.88" y1="137.16" x2="50.8" y2="137.16" width="0.1524" layer="91"/>
-</segment>
-</net>
+<wire x1="55.88" y1="137.16" x2="53.34" y2="137.16" width="0.1524" layer="91"/>
+<pinref part="3VM" gate="G$1" pin="TP"/>
+<wire x1="53.34" y1="137.16" x2="50.8" y2="137.16" width="0.1524" layer="91"/>
+<wire x1="53.34" y1="129.54" x2="53.34" y2="137.16" width="0.1524" layer="91"/>
+<junction x="53.34" y="137.16"/>
+</segment>
+</net>
